Commit message: edited joint names for consistency

File: src/scarabot/scarabot_description/urdf/robot.urdf (robot description, URDF)
Before this commit: robot scarabot, 9 links, 8 joints
Joints:
- removed joint prismatic_arm
- removed joint revolute_cylinder1
- removed joint revolute_cylinder2
- added joint prismatic_joint: type prismatic, parent link5, child gripper_prismatic, origin xyz=0.4 0 -0.05 rpy=0 0 0, axis 0 0 1, limit lower=-0.5 upper=0.5 effort=100 velocity=0.1
- added joint revolute_joint_1: type revolute, parent baselink, child revolute_link1, origin xyz=0 0 0.3 rpy=0 0 0, axis 0 0 1, limit lower=-3.1415926535897931 upper=3.1415926535897931 effort=100 velocity=0.1
- added joint revolute_joint_2: type revolute, parent link3, child revolute_link2, origin xyz=0.6 0 -0.25 rpy=0 0 0, axis 0 0 1, limit lower=-3 upper=3 effort=100 velocity=0.1

File: src/scarabot/scarabot_description/urdf/scarabot.urdf.xacro (robot description, xacro)
@@ -182,5 +182,5 @@
   <xacro:horizontal_link number="2"/>
 <!-- * * * prismatic_joint * * * -->
-  <joint name="joint_prismatic" type="prismatic">
+  <joint name="prismatic_joint" type="prismatic">
     <axis xyz="0 0 1"/>
     <limit effort="100" lower="-0.5" upper="0.5" velocity="0.1"/>
