Commit message: Update scarabot.urdf.xacro
Turnoff the gravity and adjust the prismatic link location.

File: src/scarabot/scarabot_description/urdf/scarabot.urdf.xacro (robot description, xacro)
@@ -89,5 +89,5 @@
   <link name="prismatic_link">
     <collision>
-      <origin rpy="0 0 0" xyz="0 0 0.05"/>
+      <origin rpy="0 0 0" xyz="0 0 0"/>
       <geometry>
         <box size="0.1 0.1 0.1"/>
@@ -95,5 +95,5 @@
     </collision>
     <visual>
-       <origin rpy="0 0 0" xyz="0 0 0.05"/>
+       <origin rpy="0 0 0" xyz="0 0 0"/>
       <geometry>
         <box size="0.1 0.1 0.1"/>
@@ -101,5 +101,5 @@
     </visual>
     <inertial>
-      <origin rpy="0 0 0" xyz="0 0 0.05"/>
+      <origin rpy="0 0 0" xyz="0 0 0"/>
     <mass value="0.001"/>
     <inertia
@@ -111,4 +111,5 @@
     <gazebo reference="prismatic_link">
   <material>Gazebo/Grey</material>
+        <turnGravityOff>true</turnGravityOff>
 </gazebo>
 </xacro:macro>

Commit message: Tweaked timing, added inertia

File: src/scarabot/scarabot_description/urdf/scarabot.urdf.xacro (robot description, xacro)
@@ -1,9 +1,9 @@
 <?xml version="1.0" ?>
 <robot name="scarabot" xmlns:xacro="http://www.ros.org/wiki/xacro">
-    <gazebo>
-        <plugin name="gazebo_ros_control" filename="libgazebo_ros_control.so">
-            <robotNamespace>/scarabot</robotNamespace>
-        </plugin>
-    </gazebo>
+<!--<gazebo>-->
+<!--  <plugin name = "gazebo_ros_control" filename="libgazebo_ros_control.so"-->
+<!--          <robotNamesspace>/scara_robot</robotNamesspace>-->
+<!--  </plugin>-->
+<!--</gazebo>-->
     <!-- MACROS -->
 <xacro:property name="m" value="1" />
@@ -102,9 +102,9 @@
     <inertial>
       <origin rpy="0 0 0" xyz="0 0 0"/>
-    <mass value="0.001"/>
-    <inertia
-      ixx="0" ixy="0.0" ixz="0.0"
-      iyy="0" iyz="0.0"
-      izz="0.1"/>
+    <mass value="1.0"/>
+    <inertia
+      ixx="0.0833" ixy="0.0" ixz="0.0"
+      iyy="0.0833" iyz="0.0"
+      izz="0.0833"/>
     </inertial>
   </link>
@@ -214,9 +214,9 @@
     <inertial>
       <origin rpy="0 0 0" xyz="0 0 0"/>
-    <mass value="1"/>
-    <inertia
-      ixx="0" ixy="0.0" ixz="0.0"
-      iyy="0" iyz="0.0"
-      izz="0"/>
+      <mass value="1"/>
+      <inertia
+        ixx="0.0" ixy="0.0" ixz="0.0"
+        iyy="0.0" iyz="0.0"
+        izz="0.0"/>
     </inertial>
   </link>

Commit message: GB manual merge

File: src/scarabot/scarabot_description/urdf/scarabot.urdf.xacro (robot description, xacro)
@@ -1,9 +1,9 @@
 <?xml version="1.0" ?>
 <robot name="scarabot" xmlns:xacro="http://www.ros.org/wiki/xacro">
-<!--<gazebo>-->
-<!--  <plugin name = "gazebo_ros_control" filename="libgazebo_ros_control.so"-->
-<!--          <robotNamesspace>/scara_robot</robotNamesspace>-->
-<!--  </plugin>-->
-<!--</gazebo>-->
+<!--    <gazebo>-->
+<!--        <plugin name="gazebo_ros_control" filename="libgazebo_ros_control.so">-->
+<!--            <robotNamespace>/scarabot</robotNamespace>-->
+<!--        </plugin>-->
+<!--    </gazebo>-->
     <!-- MACROS -->
 <xacro:property name="m" value="1" />
@@ -93,4 +93,6 @@
         <box size="0.1 0.1 0.1"/>
       </geometry>
+            <surface>
+      </surface>
     </collision>
     <visual>
@@ -102,5 +104,5 @@
     <inertial>
       <origin rpy="0 0 0" xyz="0 0 0"/>
-    <mass value="1.0"/>
+    <mass value="1"/>
     <inertia
       ixx="0.0833" ixy="0.0" ixz="0.0"
@@ -139,6 +141,6 @@
   <joint name="revolute_joint_1" type="revolute">
     <axis xyz="0 0 1"/>
+    <origin rpy="0 0 0" xyz="0 0 0.6"/>
     <limit effort="100" lower="-3.1415926535897931" upper="3.1415926535897931" velocity="0.1"/>
-    <origin rpy="0 0 0" xyz="0 0 0.6"/>
     <parent link="vertical_link1"/>
     <child link="revolute_link1"/>
@@ -214,9 +216,9 @@
     <inertial>
       <origin rpy="0 0 0" xyz="0 0 0"/>
-      <mass value="1"/>
-      <inertia
-        ixx="0.0" ixy="0.0" ixz="0.0"
-        iyy="0.0" iyz="0.0"
-        izz="0.0"/>
+    <mass value="1"/>
+    <inertia
+      ixx="0" ixy="0.0" ixz="0.0"
+      iyy="0" iyz="0.0"
+      izz="0"/>
     </inertial>
   </link>
