Commit message: 12/2

File: scarabot_description/urdf/scarabot.urdf.xacro (robot description, xacro)
@@ -1,9 +1,9 @@
 <?xml version="1.0" ?>
 <robot name="scarabot" xmlns:xacro="http://www.ros.org/wiki/xacro">
-    <gazebo>
-        <plugin name="gazebo_ros_control" filename="libgazebo_ros_control.so">
-            <robotNamespace>/scarabot</robotNamespace>
-        </plugin>
-    </gazebo>
+<!--    <gazebo>-->
+<!--        <plugin name="gazebo_ros_control" filename="libgazebo_ros_control.so">-->
+<!--            <robotNamespace>/scarabot</robotNamespace>-->
+<!--        </plugin>-->
+<!--    </gazebo>-->
     <!-- MACROS -->
 <xacro:property name="m" value="1" />
@@ -93,4 +93,6 @@
         <box size="0.1 0.1 0.1"/>
       </geometry>
+            <surface>
+      </surface>
     </collision>
     <visual>
@@ -102,9 +104,9 @@
     <inertial>
       <origin rpy="0 0 0" xyz="0 0 0"/>
-    <mass value="0.001"/>
-    <inertia
-      ixx="0" ixy="0.0" ixz="0.0"
-      iyy="0" iyz="0.0"
-      izz="0.1"/>
+    <mass value="1"/>
+    <inertia
+      ixx="0.0833" ixy="0.0" ixz="0.0"
+      iyy="0.0833" iyz="0.0"
+      izz="0.0833"/>
     </inertial>
   </link>
@@ -139,6 +141,6 @@
   <joint name="revolute_joint_1" type="revolute">
     <axis xyz="0 0 1"/>
+    <origin rpy="0 0 0" xyz="0 0 0.6"/>
     <limit effort="100" lower="-3.1415926535897931" upper="3.1415926535897931" velocity="0.1"/>
-    <origin rpy="0 0 0" xyz="0 0 0.6"/>
     <parent link="vertical_link1"/>
     <child link="revolute_link1"/>

Commit message: 1,2,3 done

File: scarabot_description/urdf/scarabot.urdf.xacro (robot description, xacro)
@@ -29,9 +29,9 @@
     <inertial>
       <origin rpy="0 0 0" xyz="0 0 0.25"/>
-    <mass value="1"/>
-    <inertia
-      ixx="0" ixy="0.0" ixz="0.0"
-      iyy="0" iyz="0.0"
-      izz="0"/>
+    <mass value="0.1"/>
+    <inertia
+      ixx="0.002646" ixy="0.0" ixz="0.0"
+      iyy="0.002646" iyz="0.0"
+      izz="0.001125"/>
     </inertial>
   </link>
@@ -54,9 +54,9 @@
     <inertial>
       <origin rpy="0 0 0" xyz="0 0 0.3"/>
-    <mass value="${m}"/>
-    <inertia
-      ixx="0" ixy="0.0" ixz="0.0"
-      iyy="0" iyz="0.0"
-      izz="0"/>
+    <mass value="1"/>
+    <inertia
+      ixx="0.03013" ixy="0.0" ixz="0.0"
+      iyy="0.00026" iyz="0.0"
+      izz="0.03013"/>
     </inertial>
   </link>
@@ -80,7 +80,7 @@
     <mass value="1"/>
     <inertia
-      ixx="0" ixy="0.0" ixz="0.0"
-      iyy="0" iyz="0.0"
-      izz="0"/>
+      ixx="0.00026" ixy="0.0" ixz="0.0"
+      iyy="0.02096" iyz="0.0"
+      izz="0.02096"/>
     </inertial>
   </link>
@@ -104,9 +104,9 @@
     <inertial>
       <origin rpy="0 0 0" xyz="0 0 0"/>
-    <mass value="1"/>
-    <inertia
-      ixx="0.0833" ixy="0.0" ixz="0.0"
-      iyy="0.0833" iyz="0.0"
-      izz="0.0833"/>
+    <mass value="0.1"/>
+    <inertia
+      ixx="0.000167" ixy="0.0" ixz="0.0"
+      iyy="0.000167" iyz="0.0"
+      izz="0.000167"/>
     </inertial>
   </link>

File: scarabot_description/urdf/scarabot_y_init.urdf.xacro (robot description, xacro)
@@ -29,9 +29,9 @@
     <inertial>
       <origin rpy="0 0 0" xyz="0 0 0.25"/>
-    <mass value="1"/>
-    <inertia
-      ixx="0.0833" ixy="0.0" ixz="0.0"
-      iyy="0.0833" iyz="0.0"
-      izz="0.0833"/>
+    <mass value="0.1"/>
+    <inertia
+      ixx="0.002646" ixy="0.0" ixz="0.0"
+      iyy="0.002646" iyz="0.0"
+      izz="0.001125"/>
     </inertial>
   </link>
@@ -54,9 +54,9 @@
     <inertial>
       <origin rpy="0 0 0" xyz="0 0 0.3"/>
-    <mass value="${m}"/>
-    <inertia
-      ixx="0.0833" ixy="0.0" ixz="0.0"
-      iyy="0.0833" iyz="0.0"
-      izz="0.0833"/>
+    <mass value="1"/>
+    <inertia
+      ixx="0.03013" ixy="0.0" ixz="0.0"
+      iyy="0.00026" iyz="0.0"
+      izz="0.03013"/>
     </inertial>
   </link>
@@ -80,7 +80,7 @@
     <mass value="1"/>
     <inertia
-      ixx="0.0833" ixy="0.0" ixz="0.0"
-      iyy="0.0833" iyz="0.0"
-      izz="0.0833"/>
+      ixx="0.00026" ixy="0.0" ixz="0.0"
+      iyy="0.02096" iyz="0.0"
+      izz="0.02096"/>
     </inertial>
   </link>
@@ -104,9 +104,9 @@
     <inertial>
       <origin rpy="0 0 0" xyz="0 0 0"/>
-    <mass value="1"/>
-    <inertia
-      ixx="0.0833" ixy="0.0" ixz="0.0"
-      iyy="0.0833" iyz="0.0"
-      izz="0.0833"/>
+    <mass value="0.1"/>
+    <inertia
+      ixx="0.000167" ixy="0.0" ixz="0.0"
+      iyy="0.000167" iyz="0.0"
+      izz="0.000167"/>
     </inertial>
   </link>
@@ -141,5 +141,5 @@
   <joint name="revolute_joint_1" type="revolute">
     <axis xyz="0 0 1"/>
-    <origin rpy="0 0 0" xyz="0 0 0.6"/>
+    <origin rpy="0 0 0.779923399892" xyz="0 0 0.6"/>
     <limit effort="100" lower="-3.1415926535897931" upper="3.1415926535897931" velocity="0.1"/>
     <parent link="vertical_link1"/>
@@ -169,5 +169,5 @@
     <axis xyz="0 0 1"/>
     <limit effort="100" lower="-3" upper="3" velocity="0.1"/>
-    <origin rpy="0 0 0" xyz="0.6 0 -0.25"/>
+    <origin rpy="0 0 2.85322720915" xyz="0.6 0 -0.25"/>
     <parent link="horizontal_link1"/>
     <child link="revolute_link2"/>
